File: playLight/schematic/playLight_rev_A/playLight_rev_A.kicad_sch (KiCad schematic)
At the start: 0 parts

Commit message: added first draft of the schematic added outline for the PCB and first placement of the LEDs
Parts:
- added D1, D10, D11, D12, D2, D3, D4, D5, D6, D7, D8, D9: ASMT-YTB7-0AA02, LED_SMD:LED_Avago_PLCC6_3x2.8mm, symbol LED:ASMT-YTB7-0AA02
- added J1, J2, J3, J4, J5, J6, J7, J8: Conn_01x01, Connector_Wire:SolderWirePad_1x01_SMD_1.5x3mm, symbol Connector_Generic:Conn_01x01
- added U1: LP5036, Package_DFN_QFN:VQFN-46-1EP_5x6mm_P0.4mm_EP2.8x3.8mm, symbol Driver_LED:LP5036
Connections:
- new net: D4.1 (KB), U1.12 (OUT11)
- new net: D4.2 (KG), U1.11 (OUT10)
- new net: D4.3 (KR), U1.10 (OUT9)
- new net: D1.4 (AR), D1.5 (AG), D1.6 (AB), D10.4 (AR), D10.5 (AG), D10.6 (AB), D11.4 (AR), D11.5 (AG), D11.6 (AB), D12.4 (AR), D12.5 (AG), D12.6 (AB), D2.4 (AR), D2.5 (AG), D2.6 (AB), D3.4 (AR), D3.5 (AG), D3.6 (AB), D4.4 (AR), D4.5 (AG), D4.6 (AB), D5.4 (AR), D5.5 (AG), D5.6 (AB), D6.4 (AR), D6.5 (AG), D6.6 (AB), D7.4 (AR), D7.5 (AG), D7.6 (AB), D8.4 (AR), D8.5 (AG), D8.6 (AB), D9.4 (AR), D9.5 (AG), D9.6 (AB), J1.1 (Pin_1), J6.1 (Pin_1)
- new net: D3.1 (KB), U1.9 (OUT8)
- new net: D3.2 (KG), U1.8 (OUT7)
- new net: D3.3 (KR), U1.7 (OUT6)
- new net: D1.1 (KB), U1.3 (OUT2)
- new net: D1.2 (KG), U1.2 (OUT1)
- new net: D1.3 (KR), U1.1 (OUT0)
- new net: D7.1 (KB), U1.21 (OUT20)
- new net: D7.2 (KG), U1.20 (OUT19)
- new net: D7.3 (KR), U1.19 (OUT18)
- new net: J2.1 (Pin_1), J7.1 (Pin_1), U1.40 (VCC)
- new net: D10.1 (KB), U1.30 (OUT29)
- new net: D10.2 (KG), U1.29 (OUT28)
- new net: D10.3 (KR), U1.28 (OUT27)
- new net: D5.3 (KR), U1.13 (OUT12)
- new net: D5.2 (KG), U1.14 (OUT13)
- new net: D5.1 (KB), U1.15 (OUT14)
- new net: D6.3 (KR), U1.16 (OUT15)
- new net: D6.2 (KG), U1.17 (OUT16)
- new net: D6.1 (KB), U1.18 (OUT17)
- new net: D8.3 (KR), U1.22 (OUT21)
- new net: D8.2 (KG), U1.23 (OUT22)
- new net: D8.1 (KB), U1.24 (OUT23)
- new net: D9.3 (KR), U1.25 (OUT24)
- new net: D9.2 (KG), U1.26 (OUT25)
- new net: D9.1 (KB), U1.27 (OUT26)
- new net: D11.3 (KR), U1.31 (OUT30)
- new net: D11.2 (KG), U1.32 (OUT31)
- new net: D11.1 (KB), U1.33 (OUT32)
- new net: D12.3 (KR), U1.34 (OUT33)
- new net: D12.2 (KG), U1.35 (OUT34)
- new net: D12.1 (KB), U1.36 (OUT35)
- new net: D2.3 (KR), U1.4 (OUT3)
- new net: D2.2 (KG), U1.5 (OUT4)
- new net: D2.1 (KB), U1.6 (OUT5)
- new net GND: J3.1 (Pin_1), J8.1 (Pin_1), U1.37 (GND), U1.46 (GND), U1.47 (GND)

Commit message: added a few swaps to simplify routing
Parts:
- added J10, J9: Conn_01x01, Connector_Wire:SolderWirePad_1x01_SMD_1.5x3mm, symbol Connector_Generic:Conn_01x01
- added J11: Conn_01x05, Connector_PinHeader_2.00mm:PinHeader_1x05_P2.00mm_Horizontal, symbol Connector_Generic:Conn_01x05
- added U2: STM32F070F6Px, Package_SO:TSSOP-20_4.4x6.5mm_P0.65mm, symbol MCU_ST_STM32F0:STM32F070F6Px
Connections:
- net GND: now also U2.15 (VSS)
- net at D4.1 (KB): now also U1.9 (OUT8); no longer U1.12 (OUT11)
- net at D4.2 (KG): now also U1.8 (OUT7); no longer U1.11 (OUT10)
- net at D4.3 (KR): now also U1.7 (OUT6); no longer U1.10 (OUT9)
- net at D3.1 (KB): now also U1.12 (OUT11); no longer U1.9 (OUT8)
- net at D3.2 (KG): now also U1.11 (OUT10); no longer U1.8 (OUT7)
- net at D3.3 (KR): now also U1.10 (OUT9); no longer U1.7 (OUT6)
- net at D1.1 (KB): now also U1.6 (OUT5); no longer U1.3 (OUT2)
- net at D1.2 (KG): now also U1.5 (OUT4); no longer U1.2 (OUT1)
- net at D1.3 (KR): now also U1.4 (OUT3); no longer U1.1 (OUT0)
- net at D7.1 (KB): now also U1.24 (OUT23); no longer U1.21 (OUT20)
- net at D7.2 (KG): now also U1.23 (OUT22); no longer U1.20 (OUT19)
- net at D7.3 (KR): now also U1.22 (OUT21); no longer U1.19 (OUT18)
- net at J2.1 (Pin_1), J7.1 (Pin_1), U1.40 (VCC): now also U2.16 (VDD), U2.5 (VDDA)
- net at D10.1 (KB): now also U1.27 (OUT26); no longer U1.30 (OUT29)
- net at D10.2 (KG): now also U1.26 (OUT25); no longer U1.29 (OUT28)
- net at D10.3 (KR): now also U1.25 (OUT24); no longer U1.28 (OUT27)
- net at D8.3 (KR): now also U1.19 (OUT18); no longer U1.22 (OUT21)
- net at D8.2 (KG): now also U1.20 (OUT19); no longer U1.23 (OUT22)
- net at D8.1 (KB): now also U1.21 (OUT20); no longer U1.24 (OUT23)
- net at D9.3 (KR): now also U1.28 (OUT27); no longer U1.25 (OUT24)
- net at D9.2 (KG): now also U1.29 (OUT28); no longer U1.26 (OUT25)
- net at D9.1 (KB): now also U1.30 (OUT29); no longer U1.27 (OUT26)
- net at U1.31 (OUT30): now also D12.3 (KR); no longer D11.3 (KR)
- net at U1.32 (OUT31): now also D12.2 (KG); no longer D11.2 (KG)
- net at U1.33 (OUT32): now also D12.1 (KB); no longer D11.1 (KB)
- net at U1.34 (OUT33): now also D11.3 (KR); no longer D12.3 (KR)
- net at U1.35 (OUT34): now also D11.2 (KG); no longer D12.2 (KG)
- net at U1.36 (OUT35): now also D11.1 (KB); no longer D12.1 (KB)
- net at D2.3 (KR): now also U1.1 (OUT0); no longer U1.4 (OUT3)
- net at D2.2 (KG): now also U1.2 (OUT1); no longer U1.5 (OUT4)
- net at D2.1 (KB): now also U1.3 (OUT2); no longer U1.6 (OUT5)
Other:
- moved on the sheet: D1, D10, D11, D12, D2, D3, D4, D7, D8, D9, J1, J2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
